Commit message: Make frame locations match Ouster manual

File: ouster_description/urdf/OS0-32.urdf.xacro (robot description, xacro)
@@ -29,8 +29,9 @@
       </collision>
     </link>
+    <!-- The "sensor frame" is centered at the bottom of the sensor body with x pointing forward away from the plug (see Ouster user manaual (https://data.ouster.io/downloads/software-user-manual/software-user-manual-v2p0.pdf#e))-->
     <joint name="${name}_baseplate_to_body" type="fixed">
       <parent link="${name}_baseplate"/>
       <child link="${name}"/>
-      <origin xyz="0 0 0.042" rpy="0 0 0" />
+      <origin xyz="0 0 0.008" rpy="0 0 0" />
     </joint>
     <link name="${name}">
@@ -48,8 +49,7 @@
       </collision>
       <visual name="base_visual">
-         <origin xyz="0 0 0.0" rpy="0 0 1.5707" />
+         <origin xyz="0 0 0.03618" rpy="0 0 1.5707" />
          <geometry>
 	         <mesh filename="package://ouster_description/meshes/os1_64.dae" />
-           <!-- <cylinder length="0.073" radius="0.04" /> -->
          </geometry>
       </visual>
@@ -57,4 +57,5 @@
     <link name="${imu_link}" />
     <link name="${lidar_link}" />
+    <!-- The Ouster driver publishes these joints, however, we must define them here for Gazebo and Robot State Publisher -->
     <joint name="${name}_imu_link_joint" type="fixed">
       <parent link="${name}" />
@@ -64,8 +65,9 @@
     <gazebo reference="${imu_link}">
     </gazebo>
+    <!-- The lidar frame points backwards towards the sensor plug and is vertical centered in the lidar window -->
     <joint name="${name}_lidar_link_joint" type="fixed">
       <parent link="${name}" />
       <child link="${lidar_link}" />
-      <origin xyz="0.0 0.0 0.03618" rpy="0 0 0" />
+      <origin xyz="0 0 0.03618" rpy="0 0 ${M_PI}" />
     </joint>
     <!-- Gazebo requires the ouster_gazebo_plugins package -->

File: ouster_description/urdf/OS1-64.urdf.xacro (robot description, xacro)
@@ -29,8 +29,9 @@
       </collision>
     </link>
+    <!-- The "sensor frame" is centered at the bottom of the sensor body with x pointing forward away from the plug (see Ouster user manaual (https://data.ouster.io/downloads/software-user-manual/software-user-manual-v2p0.pdf#e))-->
     <joint name="${name}_baseplate_to_body" type="fixed">
       <parent link="${name}_baseplate"/>
       <child link="${name}"/>
-      <origin xyz="0 0 0.042" rpy="0 0 0" />
+      <origin xyz="0 0 0.008" rpy="0 0 0" />
     </joint>
     <link name="${name}">
@@ -48,8 +49,7 @@
       </collision>
       <visual name="base_visual">
-         <origin xyz="0 0 0.0" rpy="0 0 1.5707" />
+         <origin xyz="0 0 0.03618" rpy="0 0 1.5707" />
          <geometry>
 	         <mesh filename="package://ouster_description/meshes/os1_64.dae" />
-           <!-- <cylinder length="0.073" radius="0.04" /> -->
          </geometry>
       </visual>
@@ -57,4 +57,5 @@
     <link name="${imu_link}" />
     <link name="${lidar_link}" />
+    <!-- The Ouster driver publishes these joints, however, we must define them here for Gazebo and Robot State Publisher -->
     <joint name="${name}_imu_link_joint" type="fixed">
       <parent link="${name}" />
@@ -64,8 +65,9 @@
     <gazebo reference="${imu_link}">
     </gazebo>
+    <!-- The lidar frame points backwards towards the sensor plug and is vertical centered in the lidar window -->
     <joint name="${name}_lidar_link_joint" type="fixed">
       <parent link="${name}" />
       <child link="${lidar_link}" />
-      <origin xyz="0.0 0.0 0.03618" rpy="0 0 0" />
+      <origin xyz="0 0 0.03618" rpy="0 0 ${M_PI}" />
     </joint>
     <!-- Gazebo requires the ouster_gazebo_plugins package -->

Commit message: Fix URDF formatting and synchronize topic names

File: ouster_description/urdf/OS0-32.urdf.xacro (robot description, xacro)
@@ -2,5 +2,5 @@
 <robot xmlns:xacro="http://www.ros.org/wiki/xacro" name="OS0-32">
   <xacro:property name="M_PI" value="3.1415926535897931" />
-  <xacro:macro name="OS0-32" params="*origin parent:=base_link name:=os0_sensor topic_points:=/os0_cloud_node/points topic_imu:=/os0_cloud_node/imu hz:=10 lasers:=32 samples:=512 min_range:=0.9 max_range:=75.0 noise:=0.008 min_angle:=-${M_PI} max_angle:=${M_PI} lidar_link:=os0_lidar imu_link:=os0_imu vfov_min:=-0.785398 vfov_max:=0.785398">
+  <xacro:macro name="OS0-32" params="*origin parent:=base_link name:=os0_sensor topic_points:=/ouster/points topic_imu:=/ouster/imu hz:=10 lasers:=32 samples:=512 min_range:=0.9 max_range:=75.0 noise:=0.008 min_angle:=-${M_PI} max_angle:=${M_PI} lidar_link:=os0_lidar imu_link:=os0_imu vfov_min:=-0.785398 vfov_max:=0.785398">
     <joint name="${name}_mount_joint" type="fixed">
       <xacro:insert_block name="origin" />
@@ -37,20 +37,20 @@
     <link name="${name}">
       <inertial>
-         <mass value="0.33"/>
-         <origin xyz="0 0 0.0365" rpy="0 0 0" />
-         <inertia ixx="0.000241148" ixy="0" ixz="0"
-          iyy="0.000241148" iyz="0" izz="0.000264"/>
+        <mass value="0.33"/>
+        <origin xyz="0 0 0.0365" rpy="0 0 0" />
+        <inertia ixx="0.000241148" ixy="0" ixz="0"
+                 iyy="0.000241148" iyz="0" izz="0.000264"/>
       </inertial>
       <collision name="base_collision">
-         <origin xyz="0 0 0.0365" rpy="0 0 0" />
-         <geometry>
+        <origin xyz="0 0 0.0365" rpy="0 0 0" />
+        <geometry>
  	        <cylinder radius="0.04" length="0.073"/>
-         </geometry>
+        </geometry>
       </collision>
       <visual name="base_visual">
-         <origin xyz="0 0 0.03618" rpy="0 0 1.5707" />
-         <geometry>
-	         <mesh filename="package://ouster_description/meshes/os1_64.dae" />
-         </geometry>
+        <origin xyz="0 0 0.03618" rpy="0 0 1.5707" />
+        <geometry>
+          <mesh filename="package://ouster_description/meshes/os1_64.dae" />
+        </geometry>
       </visual>
     </link>
@@ -73,53 +73,53 @@
     <!-- Gazebo requires the ouster_gazebo_plugins package -->
     <gazebo reference="${name}">
-        <sensor type="ray" name="${name}-OS0-32">
-          <pose>0 0 0 0 0 0</pose>
-          <visualize>false</visualize>
-          <update_rate>${hz}</update_rate>
-          <ray>
-            <scan>
-              <horizontal>
-                <samples>${samples}</samples>
-                <resolution>1</resolution>
-                <min_angle>${min_angle}</min_angle>
-                <max_angle>${max_angle}</max_angle>
-              </horizontal>
-              <vertical>
-                <samples>${lasers}</samples>
-                <resolution>1</resolution>
-                <min_angle>${vfov_min}</min_angle>
-                <max_angle>${vfov_max}</max_angle>
-              </vertical>
-            </scan>
-            <range>
-              <min>${min_range}</min>
-              <max>${max_range}</max>
-              <resolution>0.03</resolution>
-            </range>
-          </ray>
-          <plugin name="gazebo_ros_laser_controller" filename="libgazebo_ros_ouster_laser.so">
-            <topicName>${topic_points}</topicName>
-            <frameName>${lidar_link}</frameName>
-            <min_range>${min_range}</min_range>
-            <max_range>${max_range}</max_range>
-            <gaussianNoise>${noise}</gaussianNoise>
-          </plugin>
-        </sensor>
+      <sensor type="ray" name="${name}-OS0-32">
+        <pose>0 0 0 0 0 0</pose>
+        <visualize>false</visualize>
+        <update_rate>${hz}</update_rate>
+        <ray>
+          <scan>
+            <horizontal>
+              <samples>${samples}</samples>
+              <resolution>1</resolution>
+              <min_angle>${min_angle}</min_angle>
+              <max_angle>${max_angle}</max_angle>
+            </horizontal>
+            <vertical>
+              <samples>${lasers}</samples>
+              <resolution>1</resolution>
+              <min_angle>${vfov_min}</min_angle>
+              <max_angle>${vfov_max}</max_angle>
+            </vertical>
+          </scan>
+          <range>
+            <min>${min_range}</min>
+            <max>${max_range}</max>
+            <resolution>0.03</resolution>
+          </range>
+        </ray>
+        <plugin name="gazebo_ros_laser_controller" filename="libgazebo_ros_ouster_laser.so">
+          <topicName>${topic_points}</topicName>
+          <frameName>${lidar_link}</frameName>
+          <min_range>${min_range}</min_range>
+          <max_range>${max_range}</max_range>
+          <gaussianNoise>${noise}</gaussianNoise>
+        </plugin>
+      </sensor>
     </gazebo>
     <!-- IMU -->
-  <gazebo>
-    <plugin name="imu_controller" filename="libhector_gazebo_ros_imu.so">
-      <robotNamespace>/</robotNamespace>
-      <updateRate>100.0</updateRate>
-      <bodyName>${imu_link}</bodyName>
-      <topicName>${topic_imu}</topicName>
-      <accelDrift>0.005 0.005 0.005</accelDrift>
-      <accelGaussianNoise>0.005 0.005 0.005</accelGaussianNoise>
-      <rateDrift>0.005 0.005 0.005 </rateDrift>
-      <rateGaussianNoise>0.005 0.005 0.005 </rateGaussianNoise>
-      <headingDrift>0.005</headingDrift>
-      <headingGaussianNoise>0.005</headingGaussianNoise>
-    </plugin>
-  </gazebo>
+    <gazebo>
+      <plugin name="imu_controller" filename="libhector_gazebo_ros_imu.so">
+        <robotNamespace>/</robotNamespace>
+        <updateRate>100.0</updateRate>
+        <bodyName>${imu_link}</bodyName>
+        <topicName>${topic_imu}</topicName>
+        <accelDrift>0.005 0.005 0.005</accelDrift>
+        <accelGaussianNoise>0.005 0.005 0.005</accelGaussianNoise>
+        <rateDrift>0.005 0.005 0.005 </rateDrift>
+        <rateGaussianNoise>0.005 0.005 0.005 </rateGaussianNoise>
+        <headingDrift>0.005</headingDrift>
+        <headingGaussianNoise>0.005</headingGaussianNoise>
+      </plugin>
+    </gazebo>
   </xacro:macro>
 </robot>

File: ouster_description/urdf/OS1-64.urdf.xacro (robot description, xacro)
@@ -2,5 +2,5 @@
 <robot xmlns:xacro="http://www.ros.org/wiki/xacro" name="OS1-64">
   <xacro:property name="M_PI" value="3.1415926535897931" />
-  <xacro:macro name="OS1-64" params="*origin parent:=base_link name:=os_sensor topic_points:=/ouster/points topic_imu:=/ouster/imu hz:=10 lasers:=64 samples:=512 min_range:=0.9 max_range:=75.0 noise:=0.008 min_angle:=-${M_PI} max_angle:=${M_PI} lidar_link:=os_lidar imu_link:=os_imu vfov_min:=-.26 vfov_max:=.26">
+  <xacro:macro name="OS1-64" params="*origin parent:=base_link name:=os1_sensor topic_points:=/ouster/points topic_imu:=/ouster/imu hz:=10 lasers:=64 samples:=512 min_range:=0.9 max_range:=75.0 noise:=0.008 min_angle:=-${M_PI} max_angle:=${M_PI} lidar_link:=os1_lidar imu_link:=os1_imu vfov_min:=-.26 vfov_max:=.26">
     <joint name="${name}_mount_joint" type="fixed">
       <xacro:insert_block name="origin" />
@@ -37,20 +37,20 @@
     <link name="${name}">
       <inertial>
-         <mass value="0.33"/>
-         <origin xyz="0 0 0.0365" rpy="0 0 0" />
-         <inertia ixx="0.000241148" ixy="0" ixz="0"
-          iyy="0.000241148" iyz="0" izz="0.000264"/>
+        <mass value="0.33"/>
+        <origin xyz="0 0 0.0365" rpy="0 0 0" />
+        <inertia ixx="0.000241148" ixy="0" ixz="0"
+                 iyy="0.000241148" iyz="0" izz="0.000264"/>
       </inertial>
       <collision name="base_collision">
-         <origin xyz="0 0 0.0365" rpy="0 0 0" />
-         <geometry>
+        <origin xyz="0 0 0.0365" rpy="0 0 0" />
+        <geometry>
  	        <cylinder radius="0.04" length="0.073"/>
-         </geometry>
+        </geometry>
       </collision>
       <visual name="base_visual">
-         <origin xyz="0 0 0.03618" rpy="0 0 1.5707" />
-         <geometry>
-	         <mesh filename="package://ouster_description/meshes/os1_64.dae" />
-         </geometry>
+        <origin xyz="0 0 0.03618" rpy="0 0 1.5707" />
+        <geometry>
+	        <mesh filename="package://ouster_description/meshes/os1_64.dae" />
+        </geometry>
       </visual>
     </link>
@@ -63,6 +63,4 @@
       <origin xyz="0.006253 -0.011775 0.007645" rpy="0 0 0" />
     </joint>
-    <gazebo reference="${imu_link}">
-    </gazebo>
     <!-- The lidar frame points backwards towards the sensor plug and is vertical centered in the lidar window -->
     <joint name="${name}_lidar_link_joint" type="fixed">
@@ -73,53 +71,53 @@
     <!-- Gazebo requires the ouster_gazebo_plugins package -->
     <gazebo reference="${name}">
-        <sensor type="ray" name="${name}-OS1-64">
-          <pose>0 0 0 0 0 0</pose>
-          <visualize>false</visualize>
-          <update_rate>${hz}</update_rate>
-          <ray>
-            <scan>
-              <horizontal>
-                <samples>${samples}</samples>
-                <resolution>1</resolution>
-                <min_angle>${min_angle}</min_angle>
-                <max_angle>${max_angle}</max_angle>
-              </horizontal>
-              <vertical>
-                <samples>${lasers}</samples>
-                <resolution>1</resolution>
-                <min_angle>${vfov_min}</min_angle>
-                <max_angle>${vfov_max}</max_angle>
-              </vertical>
-            </scan>
-            <range>
-              <min>${min_range}</min>
-              <max>${max_range}</max>
-              <resolution>0.03</resolution>
-            </range>
-          </ray>
-          <plugin name="gazebo_ros_laser_controller" filename="libgazebo_ros_ouster_laser.so">
-            <topicName>${topic_points}</topicName>
-            <frameName>${lidar_link}</frameName>
-            <min_range>${min_range}</min_range>
-            <max_range>${max_range}</max_range>
-            <gaussianNoise>${noise}</gaussianNoise>
-          </plugin>
-        </sensor>
+      <sensor type="ray" name="${name}-OS1-64">
+        <pose>0 0 0 0 0 0</pose>
+        <visualize>false</visualize>
+        <update_rate>${hz}</update_rate>
+        <ray>
+          <scan>
+            <horizontal>
+              <samples>${samples}</samples>
+              <resolution>1</resolution>
+              <min_angle>${min_angle}</min_angle>
+              <max_angle>${max_angle}</max_angle>
+            </horizontal>
+            <vertical>
+              <samples>${lasers}</samples>
+              <resolution>1</resolution>
+              <min_angle>${vfov_min}</min_angle>
+              <max_angle>${vfov_max}</max_angle>
+            </vertical>
+          </scan>
+          <range>
+            <min>${min_range}</min>
+            <max>${max_range}</max>
+            <resolution>0.03</resolution>
+          </range>
+        </ray>
+        <plugin name="gazebo_ros_laser_controller" filename="libgazebo_ros_ouster_laser.so">
+          <topicName>${topic_points}</topicName>
+          <frameName>${lidar_link}</frameName>
+          <min_range>${min_range}</min_range>
+          <max_range>${max_range}</max_range>
+          <gaussianNoise>${noise}</gaussianNoise>
+        </plugin>
+      </sensor>
     </gazebo>
     <!-- IMU -->
-  <gazebo>
-    <plugin name="imu_controller" filename="libhector_gazebo_ros_imu.so">
-      <robotNamespace>/</robotNamespace>
-      <updateRate>100.0</updateRate>
-      <bodyName>${imu_link}</bodyName>
-      <topicName>${topic_imu}</topicName>
-      <accelDrift>0.005 0.005 0.005</accelDrift>
-      <accelGaussianNoise>0.005 0.005 0.005</accelGaussianNoise>
-      <rateDrift>0.005 0.005 0.005 </rateDrift>
-      <rateGaussianNoise>0.005 0.005 0.005 </rateGaussianNoise>
-      <headingDrift>0.005</headingDrift>
-      <headingGaussianNoise>0.005</headingGaussianNoise>
-    </plugin>
-  </gazebo>
+    <gazebo>
+      <plugin name="imu_controller" filename="libhector_gazebo_ros_imu.so">
+        <robotNamespace>/</robotNamespace>
+        <updateRate>100.0</updateRate>
+        <bodyName>${imu_link}</bodyName>
+        <topicName>${topic_imu}</topicName>
+        <accelDrift>0.005 0.005 0.005</accelDrift>
+        <accelGaussianNoise>0.005 0.005 0.005</accelGaussianNoise>
+        <rateDrift>0.005 0.005 0.005 </rateDrift>
+        <rateGaussianNoise>0.005 0.005 0.005 </rateGaussianNoise>
+        <headingDrift>0.005</headingDrift>
+        <headingGaussianNoise>0.005</headingGaussianNoise>
+      </plugin>
+    </gazebo>
   </xacro:macro>
 </robot>

Commit message: Make Ouster macros configurable between Rev6-7
Rev7 sensors are a little taller.

File: ouster_description/urdf/OS0-32.urdf.xacro (robot description, xacro)
@@ -2,5 +2,13 @@
 <robot xmlns:xacro="http://www.ros.org/wiki/xacro" name="OS0-32">
   <xacro:property name="M_PI" value="3.1415926535897931" />
-  <xacro:macro name="OS0-32" params="*origin parent:=base_link name:=os0_sensor topic_points:=/ouster/points topic_imu:=/ouster/imu hz:=10 lasers:=32 samples:=512 min_range:=0.9 max_range:=75.0 noise:=0.008 min_angle:=-${M_PI} max_angle:=${M_PI} lidar_link:=os0_lidar imu_link:=os0_imu vfov_min:=-0.785398 vfov_max:=0.785398">
+  <xacro:property name="rev6_lidar_z" value="0.03622"/>
+  <xacro:property name="rev7_lidar_z" value="0.038195"/>
+  <xacro:macro name="OS0-32" params="rev:=rev6 *origin parent:=base_link name:=os0_sensor topic_points:=/ouster/points topic_imu:=/ouster/imu hz:=10 lasers:=32 samples:=512 min_range:=0.9 max_range:=75.0 noise:=0.008 min_angle:=-${M_PI} max_angle:=${M_PI} lidar_link:=os0_lidar imu_link:=os0_imu vfov_min:=-0.785398 vfov_max:=0.785398">
+    <xacro:if value="${rev == 'rev6'}">
+      <xacro:property name="lidar_z" value="${rev6_lidar_z}"/>
+    </xacro:if>
+    <xacro:if value="${rev == 'rev7'}">
+      <xacro:property name="lidar_z" value="${rev7_lidar_z}"/>
+    </xacro:if>
     <joint name="${name}_mount_joint" type="fixed">
       <xacro:insert_block name="origin" />
@@ -69,5 +77,5 @@
       <parent link="${name}" />
       <child link="${lidar_link}" />
-      <origin xyz="0 0 0.03618" rpy="0 0 ${M_PI}" />
+      <origin xyz="0 0 ${lidar_z}" rpy="0 0 ${M_PI}" />
     </joint>
     <!-- Gazebo requires the ouster_gazebo_plugins package -->

File: ouster_description/urdf/OS1-64.urdf.xacro (robot description, xacro)
@@ -2,5 +2,13 @@
 <robot xmlns:xacro="http://www.ros.org/wiki/xacro" name="OS1-64">
   <xacro:property name="M_PI" value="3.1415926535897931" />
-  <xacro:macro name="OS1-64" params="*origin parent:=base_link name:=os1_sensor topic_points:=/ouster/points topic_imu:=/ouster/imu hz:=10 lasers:=64 samples:=512 min_range:=0.9 max_range:=75.0 noise:=0.008 min_angle:=-${M_PI} max_angle:=${M_PI} lidar_link:=os1_lidar imu_link:=os1_imu vfov_min:=-.26 vfov_max:=.26">
+  <xacro:property name="rev6_lidar_z" value="0.03622"/>
+  <xacro:property name="rev7_lidar_z" value="0.038195"/>
+  <xacro:macro name="OS1-64" params="rev:=rev6 *origin parent:=base_link name:=os1_sensor topic_points:=/ouster/points topic_imu:=/ouster/imu hz:=10 lasers:=64 samples:=512 min_range:=0.9 max_range:=75.0 noise:=0.008 min_angle:=-${M_PI} max_angle:=${M_PI} lidar_link:=os1_lidar imu_link:=os1_imu vfov_min:=-.26 vfov_max:=.26">
+    <xacro:if value="${rev == 'rev6'}">
+      <xacro:property name="lidar_z" value="${rev6_lidar_z}"/>
+    </xacro:if>
+    <xacro:if value="${rev == 'rev7'}">
+      <xacro:property name="lidar_z" value="${rev7_lidar_z}"/>
+    </xacro:if>
     <joint name="${name}_mount_joint" type="fixed">
       <xacro:insert_block name="origin" />
@@ -67,5 +75,5 @@
       <parent link="${name}" />
       <child link="${lidar_link}" />
-      <origin xyz="0 0 0.03618" rpy="0 0 ${M_PI}" />
+      <origin xyz="0 0 ${lidar_z}" rpy="0 0 ${M_PI}" />
     </joint>
     <!-- Gazebo requires the ouster_gazebo_plugins package -->
